Commit message: Gazebo-Advancements for HUD and Environements

File: ControlSystemsPipeline/tranq_ws/src/tranq_description/urdf/drone.urdf.xacro (robot description, xacro)
@@ -1,32 +1,8 @@
 <?xml version="1.0"?>
 <robot xmlns:xacro="http://www.ros.org/wiki/xacro" name="tranq_drone">
+  <xacro:include filename="$(find tranq_description)/urdf/base.urdf.xacro"/>
   <xacro:include filename="$(find tranq_description)/urdf/sensors.urdf.xacro"/>
-  <link name="base_link">
-    <inertial>
-      <origin xyz="0 0 0" rpy="0 0 0"/>
-      <mass value="1.5"/>
-      <inertia ixx="0.03" ixy="0.0" ixz="0.0" iyy="0.03" iyz="0.0" izz="0.05"/>
-    </inertial>
-    <visual>
-      <origin xyz="0 0 0" rpy="0 0 0"/>
-      <geometry><box size="0.35 0.35 0.08"/></geometry>
-      <material name="dark_grey"><color rgba="0.2 0.2 0.2 1"/></material>
-    </visual>
-    <collision>
-      <origin xyz="0 0 0" rpy="0 0 0"/>
-      <geometry><box size="0.35 0.35 0.08"/></geometry>
-    </collision>
-  </link>
   <xacro:camera_sensor parent="base_link"/>
-  <xacro:tof_sensor parent="base_link"
-    name="tof_center" topic="/range_1"
-    xyz="0.15 0.0 -0.02" rpy="0 1.5708 0"/>
-  <xacro:tof_sensor parent="base_link"
-    name="tof_offset" topic="/range_2"
-    xyz="0.15 0.0 -0.12" rpy="0 1.5708 0"/>
-  <gazebo>
-    <plugin name="gazebo_ros_control" filename="libgazebo_ros_control.so">
-      <robotNamespace>/tranq_drone</robotNamespace>
-    </plugin>
-  </gazebo>
+  <xacro:tof_sensor parent="base_link" name="tof_center" topic="/range_1" xyz="0.18 0.0 -0.02" rpy="0 1.5708 0"/>
+  <xacro:tof_sensor parent="base_link" name="tof_offset" topic="/range_2" xyz="0.18 0.0 -0.12" rpy="0 1.5708 0"/>
 </robot>

Commit message: added the missing files

File: ControlSystemsPipeline/tranq_ws/src/tranq_description/urdf/drone.urdf.xacro (robot description, xacro)
@@ -1,8 +1,207 @@
 <?xml version="1.0"?>
 <robot xmlns:xacro="http://www.ros.org/wiki/xacro" name="tranq_drone">
-  <xacro:include filename="$(find tranq_description)/urdf/base.urdf.xacro"/>
-  <xacro:include filename="$(find tranq_description)/urdf/sensors.urdf.xacro"/>
-  <xacro:camera_sensor parent="base_link"/>
-  <xacro:tof_sensor parent="base_link" name="tof_center" topic="/range_1" xyz="0.18 0.0 -0.02" rpy="0 1.5708 0"/>
-  <xacro:tof_sensor parent="base_link" name="tof_offset" topic="/range_2" xyz="0.18 0.0 -0.12" rpy="0 1.5708 0"/>
+  <!-- ── Materials ─────────────────────────────────────────── -->
+  <material name="dark_grey"><color rgba="0.15 0.15 0.15 1.0"/></material>
+  <material name="orange">   <color rgba="0.9  0.4  0.0  1.0"/></material>
+  <material name="black">    <color rgba="0.05 0.05 0.05 1.0"/></material>
+  <!-- ── Base link (central body) ──────────────────────────── -->
+  <link name="base_link">
+    <inertial>
+      <mass value="2.5"/>
+      <origin xyz="0 0 0" rpy="0 0 0"/>
+      <inertia ixx="0.04" ixy="0.0" ixz="0.0"
+               iyy="0.04" iyz="0.0" izz="0.07"/>
+    </inertial>
+    <visual>
+      <origin xyz="0 0 0" rpy="0 0 0.785"/>
+      <geometry><box size="0.38 0.10 0.07"/></geometry>
+      <material name="dark_grey"/>
+    </visual>
+    <visual>
+      <origin xyz="0 0 0" rpy="0 0 -0.785"/>
+      <geometry><box size="0.38 0.10 0.07"/></geometry>
+      <material name="dark_grey"/>
+    </visual>
+    <!-- Central hub -->
+    <visual>
+      <origin xyz="0 0 0.02" rpy="0 0 0"/>
+      <geometry><cylinder radius="0.07" length="0.06"/></geometry>
+      <material name="orange"/>
+    </visual>
+    <collision>
+      <origin xyz="0 0 0" rpy="0 0 0"/>
+      <geometry><box size="0.55 0.55 0.12"/></geometry>
+    </collision>
+  </link>
+  <!-- ── 4 Motor + Prop visual links ───────────────────────── -->
+  <xacro:macro name="motor_link" params="name x y">
+    <link name="${name}">
+      <visual>
+        <origin xyz="0 0 0.025" rpy="0 0 0"/>
+        <geometry><cylinder radius="0.025" length="0.06"/></geometry>
+        <material name="black"/>
+      </visual>
+      <!-- Prop disk -->
+      <visual>
+        <origin xyz="0 0 0.06" rpy="0 0 0"/>
+        <geometry><cylinder radius="0.115" length="0.004"/></geometry>
+        <material name="dark_grey"/>
+      </visual>
+    </link>
+    <joint name="${name}_joint" type="fixed">
+      <parent link="base_link"/>
+      <child  link="${name}"/>
+      <origin xyz="${x} ${y} 0.02" rpy="0 0 0"/>
+    </joint>
+  </xacro:macro>
+  <xacro:motor_link name="motor_fl" x=" 0.22" y=" 0.22"/>
+  <xacro:motor_link name="motor_fr" x=" 0.22" y="-0.22"/>
+  <xacro:motor_link name="motor_rl" x="-0.22" y=" 0.22"/>
+  <xacro:motor_link name="motor_rr" x="-0.22" y="-0.22"/>
+  <!-- ── Landing legs ──────────────────────────────────────── -->
+  <xacro:macro name="leg" params="name x y">
+    <link name="${name}">
+      <visual>
+        <origin xyz="0 0 -0.07" rpy="0 0 0"/>
+        <geometry><cylinder radius="0.008" length="0.14"/></geometry>
+        <material name="dark_grey"/>
+      </visual>
+    </link>
+    <joint name="${name}_joint" type="fixed">
+      <parent link="base_link"/>
+      <child  link="${name}"/>
+      <origin xyz="${x} ${y} -0.04" rpy="0 0 0"/>
+    </joint>
+  </xacro:macro>
+  <xacro:leg name="leg_fl" x=" 0.15" y=" 0.15"/>
+  <xacro:leg name="leg_fr" x=" 0.15" y="-0.15"/>
+  <xacro:leg name="leg_rl" x="-0.15" y=" 0.15"/>
+  <xacro:leg name="leg_rr" x="-0.15" y="-0.15"/>
+  <!-- ── Camera gimbal + sensor ────────────────────────────── -->
+  <link name="gimbal_link">
+    <visual>
+      <origin xyz="0 0 0" rpy="0 0 0"/>
+      <geometry><box size="0.06 0.06 0.05"/></geometry>
+      <material name="black"/>
+    </visual>
+  </link>
+  <joint name="gimbal_joint" type="fixed">
+    <parent link="base_link"/>
+    <child  link="gimbal_link"/>
+    <origin xyz="0.16 0.0 -0.05" rpy="0 0 0"/>
+  </joint>
+  <link name="camera_link"/>
+  <joint name="camera_joint" type="fixed">
+    <parent link="gimbal_link"/>
+    <child  link="camera_link"/>
+    <origin xyz="0.02 0.0 -0.03" rpy="0 ${pi/2} 0"/>
+  </joint>
+  <!-- ── ToF sensors ───────────────────────────────────────── -->
+  <link name="tof_center">
+    <visual>
+      <origin xyz="0 0 0" rpy="0 0 0"/>
+      <geometry><box size="0.02 0.02 0.01"/></geometry>
+      <material name="orange"/>
+    </visual>
+  </link>
+  <joint name="tof_center_joint" type="fixed">
+    <parent link="base_link"/>
+    <child  link="tof_center"/>
+    <origin xyz="0.0 0.0 -0.05" rpy="0 ${pi} 0"/>
+  </joint>
+  <link name="tof_offset">
+    <visual>
+      <origin xyz="0 0 0" rpy="0 0 0"/>
+      <geometry><box size="0.02 0.02 0.01"/></geometry>
+      <material name="orange"/>
+    </visual>
+  </link>
+  <joint name="tof_offset_joint" type="fixed">
+    <parent link="base_link"/>
+    <child  link="tof_offset"/>
+    <origin xyz="0.12 0.0 -0.05" rpy="0 ${pi} 0"/>
+  </joint>
+  <!-- ── Gazebo: camera plugin ─────────────────────────────── -->
+  <gazebo reference="camera_link">
+    <sensor name="tranq_camera" type="camera">
+      <always_on>true</always_on>
+      <update_rate>30</update_rate>
+      <camera>
+        <horizontal_fov>1.396</horizontal_fov>
+        <image><width>640</width><height>480</height><format>R8G8B8</format></image>
+        <clip><near>0.05</near><far>200</far></clip>
+      </camera>
+      <plugin name="camera_controller" filename="libgz-sim-sensors-system.so">
+        <ros>
+          <namespace>/</namespace>
+          <remapping>image_raw:=/camera/image_raw</remapping>
+          <remapping>camera_info:=/camera/camera_info</remapping>
+        </ros>
+      </plugin>
+    </sensor>
+  </gazebo>
+  <!-- ── Gazebo: ToF sensors ───────────────────────────────── -->
+  <gazebo reference="tof_center">
+    <sensor name="tof_center_sensor" type="gpu_lidar">
+      <always_on>true</always_on>
+      <update_rate>20</update_rate>
+      <ray>
+        <scan><horizontal><samples>1</samples><min_angle>0</min_angle><max_angle>0</max_angle></horizontal></scan>
+        <range><min>0.05</min><max>30.0</max><resolution>0.001</resolution></range>
+      </ray>
+      <plugin name="tof1" filename="libgz-sim-sensors-system.so">
+        <ros><remapping>~/out:=/range_1</remapping></ros>
+      </plugin>
+    </sensor>
+  </gazebo>
+  <gazebo reference="tof_offset">
+    <sensor name="tof_offset_sensor" type="gpu_lidar">
+      <always_on>true</always_on>
+      <update_rate>20</update_rate>
+      <ray>
+        <scan><horizontal><samples>1</samples><min_angle>0</min_angle><max_angle>0</max_angle></horizontal></scan>
+        <range><min>0.05</min><max>30.0</max><resolution>0.001</resolution></range>
+      </ray>
+      <plugin name="tof2" filename="libgz-sim-sensors-system.so">
+        <ros><remapping>~/out:=/range_2</remapping></ros>
+      </plugin>
+    </sensor>
+  </gazebo>
+  <!-- ── Gazebo: velocity controller (keeps drone airborne + responds to /cmd_vel) -->
+  <gazebo>
+    <plugin filename="gz-sim-multicopter-motor-model-system"
+            name="gz::sim::systems::MulticopterMotorModel">
+      <robotNamespace>/</robotNamespace>
+      <jointName>motor_fl_joint</jointName>
+      <linkName>motor_fl</linkName>
+      <turningDirection>ccw</turningDirection>
+      <timeConstantUp>0.0125</timeConstantUp>
+      <timeConstantDown>0.025</timeConstantDown>
+      <maxRotVelocity>1100</maxRotVelocity>
+      <motorConstant>8.54858e-6</motorConstant>
+      <momentConstant>0.016</momentConstant>
+      <commandSubTopic>command/motor_speed</commandSubTopic>
+      <motorNumber>0</motorNumber>
+      <rotorDragCoefficient>8.06428e-5</rotorDragCoefficient>
+      <rollingMomentCoefficient>1e-6</rollingMomentCoefficient>
+      <motorSpeedPubTopic>motor_speed/0</motorSpeedPubTopic>
+    </plugin>
+    <plugin filename="gz-sim-multicopter-control-system"
+            name="gz::sim::systems::MulticopterVelocityControl">
+      <robotNamespace>/</robotNamespace>
+      <commandSubTopic>cmd_vel</commandSubTopic>
+      <enableSubTopic>enable</enableSubTopic>
+      <comLinkName>base_link</comLinkName>
+      <velocityGain>2.7 2.7 2.7</velocityGain>
+      <attitudeGain>2.0 3.0 0.15</attitudeGain>
+      <angularRateGain>0.4 0.52 0.18</angularRateGain>
+      <maximumLinearAcceleration>2 2 2</maximumLinearAcceleration>
+      <rotorConfiguration>
+        <rotor><jointName>motor_fl_joint</jointName><forceConstant>8.54858e-6</forceConstant><momentConstant>0.016</momentConstant><direction>1</direction></rotor>
+        <rotor><jointName>motor_fr_joint</jointName><forceConstant>8.54858e-6</forceConstant><momentConstant>0.016</momentConstant><direction>-1</direction></rotor>
+        <rotor><jointName>motor_rl_joint</jointName><forceConstant>8.54858e-6</forceConstant><momentConstant>0.016</momentConstant><direction>-1</direction></rotor>
+        <rotor><jointName>motor_rr_joint</jointName><forceConstant>8.54858e-6</forceConstant><momentConstant>0.016</momentConstant><direction>1</direction></rotor>
+      </rotorConfiguration>
+    </plugin>
+  </gazebo>
 </robot>

Commit message: IDE for SDR files

File: ControlSystemsPipeline/tranq_ws/src/tranq_description/urdf/drone.urdf.xacro (robot description, xacro)
@@ -1,9 +1,7 @@
 <?xml version="1.0"?>
 <robot xmlns:xacro="http://www.ros.org/wiki/xacro" name="tranq_drone">
-  <!-- ── Materials ─────────────────────────────────────────── -->
   <material name="dark_grey"><color rgba="0.15 0.15 0.15 1.0"/></material>
   <material name="orange">   <color rgba="0.9  0.4  0.0  1.0"/></material>
   <material name="black">    <color rgba="0.05 0.05 0.05 1.0"/></material>
-  <!-- ── Base link (central body) ──────────────────────────── -->
   <link name="base_link">
     <inertial>
@@ -23,5 +21,4 @@
       <material name="dark_grey"/>
     </visual>
-    <!-- Central hub -->
     <visual>
       <origin xyz="0 0 0.02" rpy="0 0 0"/>
@@ -34,7 +31,12 @@
     </collision>
   </link>
-  <!-- ── 4 Motor + Prop visual links ───────────────────────── -->
+  <!-- FIX: joints are now continuous (revolute, unlimited spin) not fixed -->
   <xacro:macro name="motor_link" params="name x y">
     <link name="${name}">
+      <inertial>
+        <mass value="0.05"/>
+        <origin xyz="0 0 0" rpy="0 0 0"/>
+        <inertia ixx="1e-5" ixy="0" ixz="0" iyy="1e-5" iyz="0" izz="1e-5"/>
+      </inertial>
       <visual>
         <origin xyz="0 0 0.025" rpy="0 0 0"/>
@@ -42,5 +44,4 @@
         <material name="black"/>
       </visual>
-      <!-- Prop disk -->
       <visual>
         <origin xyz="0 0 0.06" rpy="0 0 0"/>
@@ -48,9 +49,14 @@
         <material name="dark_grey"/>
       </visual>
+      <collision>
+        <origin xyz="0 0 0.04" rpy="0 0 0"/>
+        <geometry><cylinder radius="0.115" length="0.07"/></geometry>
+      </collision>
     </link>
-    <joint name="${name}_joint" type="fixed">
+    <joint name="${name}_joint" type="continuous">
       <parent link="base_link"/>
       <child  link="${name}"/>
       <origin xyz="${x} ${y} 0.02" rpy="0 0 0"/>
+      <axis xyz="0 0 1"/>
     </joint>
   </xacro:macro>
@@ -59,5 +65,4 @@
   <xacro:motor_link name="motor_rl" x="-0.22" y=" 0.22"/>
   <xacro:motor_link name="motor_rr" x="-0.22" y="-0.22"/>
-  <!-- ── Landing legs ──────────────────────────────────────── -->
   <xacro:macro name="leg" params="name x y">
     <link name="${name}">
@@ -78,5 +83,4 @@
   <xacro:leg name="leg_rl" x="-0.15" y=" 0.15"/>
   <xacro:leg name="leg_rr" x="-0.15" y="-0.15"/>
-  <!-- ── Camera gimbal + sensor ────────────────────────────── -->
   <link name="gimbal_link">
     <visual>
@@ -97,5 +101,4 @@
     <origin xyz="0.02 0.0 -0.03" rpy="0 ${pi/2} 0"/>
   </joint>
-  <!-- ── ToF sensors ───────────────────────────────────────── -->
   <link name="tof_center">
     <visual>
@@ -122,5 +125,4 @@
     <origin xyz="0.12 0.0 -0.05" rpy="0 ${pi} 0"/>
   </joint>
-  <!-- ── Gazebo: camera plugin ─────────────────────────────── -->
   <gazebo reference="camera_link">
     <sensor name="tranq_camera" type="camera">
@@ -141,5 +143,4 @@
     </sensor>
   </gazebo>
-  <!-- ── Gazebo: ToF sensors ───────────────────────────────── -->
   <gazebo reference="tof_center">
     <sensor name="tof_center_sensor" type="gpu_lidar">
@@ -168,5 +169,4 @@
     </sensor>
   </gazebo>
-  <!-- ── Gazebo: velocity controller (keeps drone airborne + responds to /cmd_vel) -->
   <gazebo>
     <plugin filename="gz-sim-multicopter-motor-model-system"
