Commit message: fix: add MulticopterVelocityControl plugin + revolute joints + odometry publisher to drone URDF

File: ControlSystemsPipeline/tranq_ws/src/tranq_description/urdf/drone.urdf.xacro (robot description, xacro)
@@ -1,206 +1,212 @@
 <?xml version="1.0"?>
 <robot xmlns:xacro="http://www.ros.org/wiki/xacro" name="tranq_drone">
+  <!-- â”€â”€â”€ MATERIALS â”€â”€â”€ -->
   <material name="dark_grey"><color rgba="0.15 0.15 0.15 1.0"/></material>
   <material name="orange">   <color rgba="0.9  0.4  0.0  1.0"/></material>
   <material name="black">    <color rgba="0.05 0.05 0.05 1.0"/></material>
+  <!-- â”€â”€â”€ BASE LINK (FRAME) â”€â”€â”€ -->
   <link name="base_link">
     <inertial>
       <mass value="2.5"/>
       <origin xyz="0 0 0" rpy="0 0 0"/>
-      <inertia ixx="0.04" ixy="0.0" ixz="0.0"
-               iyy="0.04" iyz="0.0" izz="0.07"/>
+      <!-- Corrected inertia tensor for X-frame quadrotor: arm_len=0.25m -->
+      <inertia ixx="0.0347" ixy="0.0" ixz="0.0"
+               iyy="0.0347" iyz="0.0" izz="0.0630"/>
     </inertial>
+    <!-- X-arm 1 -->
     <visual>
       <origin xyz="0 0 0" rpy="0 0 0.785"/>
-      <geometry><box size="0.38 0.10 0.07"/></geometry>
-      <material name="dark_grey"/>
-    </visual>
+      <geometry><box size="0.50 0.08 0.06"/></geometry>
+      <material name="dark_grey"/>
+    </visual>
+    <!-- X-arm 2 -->
     <visual>
       <origin xyz="0 0 0" rpy="0 0 -0.785"/>
-      <geometry><box size="0.38 0.10 0.07"/></geometry>
-      <material name="dark_grey"/>
-    </visual>
+      <geometry><box size="0.50 0.08 0.06"/></geometry>
+      <material name="dark_grey"/>
+    </visual>
+    <!-- Center hub -->
     <visual>
       <origin xyz="0 0 0.02" rpy="0 0 0"/>
-      <geometry><cylinder radius="0.07" length="0.06"/></geometry>
+      <geometry><cylinder radius="0.09" length="0.08"/></geometry>
       <material name="orange"/>
+    </visual>
+    <!-- Dart launcher barrel -->
+    <visual>
+      <origin xyz="0.20 0 -0.04" rpy="0 1.5708 0"/>
+      <geometry><cylinder radius="0.025" length="0.18"/></geometry>
+      <material name="black"/>
+    </visual>
+    <!-- Landing legs -->
+    <visual>
+      <origin xyz=" 0.12  0.12 -0.085" rpy="0 0 0"/>
+      <geometry><cylinder radius="0.01" length="0.14"/></geometry>
+      <material name="dark_grey"/>
+    </visual>
+    <visual>
+      <origin xyz="-0.12  0.12 -0.085" rpy="0 0 0"/>
+      <geometry><cylinder radius="0.01" length="0.14"/></geometry>
+      <material name="dark_grey"/>
+    </visual>
+    <visual>
+      <origin xyz=" 0.12 -0.12 -0.085" rpy="0 0 0"/>
+      <geometry><cylinder radius="0.01" length="0.14"/></geometry>
+      <material name="dark_grey"/>
+    </visual>
+    <visual>
+      <origin xyz="-0.12 -0.12 -0.085" rpy="0 0 0"/>
+      <geometry><cylinder radius="0.01" length="0.14"/></geometry>
+      <material name="dark_grey"/>
     </visual>
     <collision>
       <origin xyz="0 0 0" rpy="0 0 0"/>
-      <geometry><box size="0.55 0.55 0.12"/></geometry>
+      <geometry><box size="0.58 0.58 0.14"/></geometry>
     </collision>
   </link>
-  <!-- FIX: joints are now continuous (revolute, unlimited spin) not fixed -->
-  <xacro:macro name="motor_link" params="name x y">
+  <!-- â”€â”€â”€ MOTOR / ROTOR MACRO â”€â”€â”€ -->
+  <!-- FIX: joints are now 'revolute' (not 'fixed') so the
+       MulticopterMotorModel plugin can apply thrust forces.
+       Previously this was 'fixed' which meant the physics
+       system saw zero rotor inertia change = no thrust. -->
+  <xacro:macro name="motor_link" params="name x y direction">
     <link name="${name}">
       <inertial>
         <mass value="0.05"/>
         <origin xyz="0 0 0" rpy="0 0 0"/>
-        <inertia ixx="1e-5" ixy="0" ixz="0" iyy="1e-5" iyz="0" izz="1e-5"/>
+        <inertia ixx="1e-5" ixy="0" ixz="0"
+                 iyy="1e-5" iyz="0" izz="9.75e-6"/>
       </inertial>
       <visual>
-        <origin xyz="0 0 0.025" rpy="0 0 0"/>
-        <geometry><cylinder radius="0.025" length="0.06"/></geometry>
+        <origin xyz="0 0 0.02" rpy="0 0 0"/>
+        <geometry><cylinder radius="0.025" length="0.05"/></geometry>
         <material name="black"/>
       </visual>
       <visual>
-        <origin xyz="0 0 0.06" rpy="0 0 0"/>
+        <origin xyz="0 0 0.055" rpy="0 0 0"/>
         <geometry><cylinder radius="0.115" length="0.004"/></geometry>
         <material name="dark_grey"/>
       </visual>
       <collision>
-        <origin xyz="0 0 0.04" rpy="0 0 0"/>
-        <geometry><cylinder radius="0.115" length="0.07"/></geometry>
+        <origin xyz="0 0 0.055" rpy="0 0 0"/>
+        <geometry><cylinder radius="0.115" length="0.01"/></geometry>
       </collision>
     </link>
-    <joint name="${name}_joint" type="continuous">
+    <joint name="${name}_joint" type="revolute">
       <parent link="base_link"/>
-      <child  link="${name}"/>
-      <origin xyz="${x} ${y} 0.02" rpy="0 0 0"/>
+      <child link="${name}"/>
+      <origin xyz="${x} ${y} 0.03" rpy="0 0 0"/>
       <axis xyz="0 0 1"/>
+      <!-- Effectively unlimited rotation for propellers -->
+      <limit lower="-1e6" upper="1e6" effort="10" velocity="3500"/>
     </joint>
+    <!-- Gz Harmonic MulticopterMotorModel plugin per rotor -->
+    <gazebo>
+      <plugin filename="gz-sim-multicopter-motor-model-system"
+              name="gz::sim::systems::MulticopterMotorModel">
+        <robotNamespace>tranq_drone</robotNamespace>
+        <jointName>${name}_joint</jointName>
+        <linkName>${name}</linkName>
+        <turningDirection>${direction}</turningDirection>
+        <timeConstantUp>0.0125</timeConstantUp>
+        <timeConstantDown>0.025</timeConstantDown>
+        <maxRotVelocity>838.0</maxRotVelocity>
+        <motorConstant>8.54858e-06</motorConstant>
+        <momentConstant>0.06</momentConstant>
+        <commandSubTopic>gazebo/command/motor_speed</commandSubTopic>
+        <motorNumber>0</motorNumber>
+        <rotorDragCoefficient>8.06428e-05</rotorDragCoefficient>
+        <rollingMomentCoefficient>1e-06</rollingMomentCoefficient>
+        <rotorVelocitySlowdownSim>10</rotorVelocitySlowdownSim>
+        <motorType>velocity</motorType>
+      </plugin>
+    </gazebo>
   </xacro:macro>
-  <xacro:motor_link name="motor_fl" x=" 0.22" y=" 0.22"/>
-  <xacro:motor_link name="motor_fr" x=" 0.22" y="-0.22"/>
-  <xacro:motor_link name="motor_rl" x="-0.22" y=" 0.22"/>
-  <xacro:motor_link name="motor_rr" x="-0.22" y="-0.22"/>
-  <xacro:macro name="leg" params="name x y">
-    <link name="${name}">
-      <visual>
-        <origin xyz="0 0 -0.07" rpy="0 0 0"/>
-        <geometry><cylinder radius="0.008" length="0.14"/></geometry>
-        <material name="dark_grey"/>
-      </visual>
-    </link>
-    <joint name="${name}_joint" type="fixed">
-      <parent link="base_link"/>
-      <child  link="${name}"/>
-      <origin xyz="${x} ${y} -0.04" rpy="0 0 0"/>
-    </joint>
-  </xacro:macro>
-  <xacro:leg name="leg_fl" x=" 0.15" y=" 0.15"/>
-  <xacro:leg name="leg_fr" x=" 0.15" y="-0.15"/>
-  <xacro:leg name="leg_rl" x="-0.15" y=" 0.15"/>
-  <xacro:leg name="leg_rr" x="-0.15" y="-0.15"/>
-  <link name="gimbal_link">
-    <visual>
-      <origin xyz="0 0 0" rpy="0 0 0"/>
-      <geometry><box size="0.06 0.06 0.05"/></geometry>
-      <material name="black"/>
-    </visual>
-  </link>
-  <joint name="gimbal_joint" type="fixed">
-    <parent link="base_link"/>
-    <child  link="gimbal_link"/>
-    <origin xyz="0.16 0.0 -0.05" rpy="0 0 0"/>
-  </joint>
-  <link name="camera_link"/>
-  <joint name="camera_joint" type="fixed">
-    <parent link="gimbal_link"/>
-    <child  link="camera_link"/>
-    <origin xyz="0.02 0.0 -0.03" rpy="0 ${pi/2} 0"/>
-  </joint>
-  <link name="tof_center">
-    <visual>
-      <origin xyz="0 0 0" rpy="0 0 0"/>
-      <geometry><box size="0.02 0.02 0.01"/></geometry>
-      <material name="orange"/>
-    </visual>
-  </link>
-  <joint name="tof_center_joint" type="fixed">
-    <parent link="base_link"/>
-    <child  link="tof_center"/>
-    <origin xyz="0.0 0.0 -0.05" rpy="0 ${pi} 0"/>
-  </joint>
-  <link name="tof_offset">
-    <visual>
-      <origin xyz="0 0 0" rpy="0 0 0"/>
-      <geometry><box size="0.02 0.02 0.01"/></geometry>
-      <material name="orange"/>
-    </visual>
-  </link>
-  <joint name="tof_offset_joint" type="fixed">
-    <parent link="base_link"/>
-    <child  link="tof_offset"/>
-    <origin xyz="0.12 0.0 -0.05" rpy="0 ${pi} 0"/>
-  </joint>
-  <gazebo reference="camera_link">
-    <sensor name="tranq_camera" type="camera">
-      <always_on>true</always_on>
-      <update_rate>30</update_rate>
-      <camera>
-        <horizontal_fov>1.396</horizontal_fov>
-        <image><width>640</width><height>480</height><format>R8G8B8</format></image>
-        <clip><near>0.05</near><far>200</far></clip>
-      </camera>
-      <plugin name="camera_controller" filename="libgz-sim-sensors-system.so">
-        <ros>
-          <namespace>/</namespace>
-          <remapping>image_raw:=/camera/image_raw</remapping>
-          <remapping>camera_info:=/camera/camera_info</remapping>
-        </ros>
-      </plugin>
-    </sensor>
-  </gazebo>
-  <gazebo reference="tof_center">
-    <sensor name="tof_center_sensor" type="gpu_lidar">
-      <always_on>true</always_on>
-      <update_rate>20</update_rate>
-      <ray>
-        <scan><horizontal><samples>1</samples><min_angle>0</min_angle><max_angle>0</max_angle></horizontal></scan>
-        <range><min>0.05</min><max>30.0</max><resolution>0.001</resolution></range>
-      </ray>
-      <plugin name="tof1" filename="libgz-sim-sensors-system.so">
-        <ros><remapping>~/out:=/range_1</remapping></ros>
-      </plugin>
-    </sensor>
-  </gazebo>
-  <gazebo reference="tof_offset">
-    <sensor name="tof_offset_sensor" type="gpu_lidar">
-      <always_on>true</always_on>
-      <update_rate>20</update_rate>
-      <ray>
-        <scan><horizontal><samples>1</samples><min_angle>0</min_angle><max_angle>0</max_angle></horizontal></scan>
-        <range><min>0.05</min><max>30.0</max><resolution>0.001</resolution></range>
-      </ray>
-      <plugin name="tof2" filename="libgz-sim-sensors-system.so">
-        <ros><remapping>~/out:=/range_2</remapping></ros>
-      </plugin>
-    </sensor>
-  </gazebo>
+  <!-- FIX: CCW on FL/RR, CW on FR/RL for correct yaw authority -->
+  <xacro:motor_link name="rotor_fl" x=" 0.177" y=" 0.177" direction="ccw"/>
+  <xacro:motor_link name="rotor_fr" x=" 0.177" y="-0.177" direction="cw"/>
+  <xacro:motor_link name="rotor_rl" x="-0.177" y=" 0.177" direction="cw"/>
+  <xacro:motor_link name="rotor_rr" x="-0.177" y="-0.177" direction="ccw"/>
+  <!-- â”€â”€â”€ INCLUDE SENSORS â”€â”€â”€ -->
+  <xacro:include filename="$(find tranq_description)/urdf/sensors.urdf.xacro"/>
+  <xacro:camera_sensor parent="base_link"/>
+  <xacro:imu_sensor parent="base_link"/>
+  <!-- â”€â”€â”€ FIX: MulticopterVelocityControl â€” THIS WAS COMPLETELY MISSING â”€â”€â”€ -->
+  <!-- This plugin translates /cmd_vel Twist into per-motor speed commands.
+       Without it the drone has no relationship between ROS velocity commands
+       and Gazebo physics â€” it simply falls through the world. -->
   <gazebo>
-    <plugin filename="gz-sim-multicopter-motor-model-system"
-            name="gz::sim::systems::MulticopterMotorModel">
-      <robotNamespace>/</robotNamespace>
-      <jointName>motor_fl_joint</jointName>
-      <linkName>motor_fl</linkName>
-      <turningDirection>ccw</turningDirection>
-      <timeConstantUp>0.0125</timeConstantUp>
-      <timeConstantDown>0.025</timeConstantDown>
-      <maxRotVelocity>1100</maxRotVelocity>
-      <motorConstant>8.54858e-6</motorConstant>
-      <momentConstant>0.016</momentConstant>
-      <commandSubTopic>command/motor_speed</commandSubTopic>
-      <motorNumber>0</motorNumber>
-      <rotorDragCoefficient>8.06428e-5</rotorDragCoefficient>
-      <rollingMomentCoefficient>1e-6</rollingMomentCoefficient>
-      <motorSpeedPubTopic>motor_speed/0</motorSpeedPubTopic>
-    </plugin>
     <plugin filename="gz-sim-multicopter-control-system"
             name="gz::sim::systems::MulticopterVelocityControl">
-      <robotNamespace>/</robotNamespace>
-      <commandSubTopic>cmd_vel</commandSubTopic>
-      <enableSubTopic>enable</enableSubTopic>
+      <robotNamespace>tranq_drone</robotNamespace>
+      <commandSubTopic>/cmd_vel</commandSubTopic>
+      <enableSubTopic>/enable_motors</enableSubTopic>
       <comLinkName>base_link</comLinkName>
       <velocityGain>2.7 2.7 2.7</velocityGain>
-      <attitudeGain>2.0 3.0 0.15</attitudeGain>
-      <angularRateGain>0.4 0.52 0.18</angularRateGain>
+      <attitudeGain>3.0 3.0 0.15</attitudeGain>
+      <angularRateGain>0.4 0.4 0.12</angularRateGain>
       <maximumLinearAcceleration>2 2 2</maximumLinearAcceleration>
-      <rotorConfiguration>
-        <rotor><jointName>motor_fl_joint</jointName><forceConstant>8.54858e-6</forceConstant><momentConstant>0.016</momentConstant><direction>1</direction></rotor>
-        <rotor><jointName>motor_fr_joint</jointName><forceConstant>8.54858e-6</forceConstant><momentConstant>0.016</momentConstant><direction>-1</direction></rotor>
-        <rotor><jointName>motor_rl_joint</jointName><forceConstant>8.54858e-6</forceConstant><momentConstant>0.016</momentConstant><direction>-1</direction></rotor>
-        <rotor><jointName>motor_rr_joint</jointName><forceConstant>8.54858e-6</forceConstant><momentConstant>0.016</momentConstant><direction>1</direction></rotor>
-      </rotorConfiguration>
+      <rotors>
+        <rotor>
+          <jointName>rotor_fl_joint</jointName>
+          <bodyFrame>rotor_fl</bodyFrame>
+          <direction>1</direction>
+          <motorConstant>8.54858e-06</motorConstant>
+          <momentConstant>0.06</momentConstant>
+          <timeConstantUp>0.0125</timeConstantUp>
+          <timeConstantDown>0.025</timeConstantDown>
+          <maxRotVelocity>838</maxRotVelocity>
+        </rotor>
+        <rotor>
+          <jointName>rotor_fr_joint</jointName>
+          <bodyFrame>rotor_fr</bodyFrame>
+          <direction>-1</direction>
+          <motorConstant>8.54858e-06</motorConstant>
+          <momentConstant>0.06</momentConstant>
+          <timeConstantUp>0.0125</timeConstantUp>
+          <timeConstantDown>0.025</timeConstantDown>
+          <maxRotVelocity>838</maxRotVelocity>
+        </rotor>
+        <rotor>
+          <jointName>rotor_rl_joint</jointName>
+          <bodyFrame>rotor_rl</bodyFrame>
+          <direction>-1</direction>
+          <motorConstant>8.54858e-06</motorConstant>
+          <momentConstant>0.06</momentConstant>
+          <timeConstantUp>0.0125</timeConstantUp>
+          <timeConstantDown>0.025</timeConstantDown>
+          <maxRotVelocity>838</maxRotVelocity>
+        </rotor>
+        <rotor>
+          <jointName>rotor_rr_joint</jointName>
+          <bodyFrame>rotor_rr</bodyFrame>
+          <direction>1</direction>
+          <motorConstant>8.54858e-06</motorConstant>
+          <momentConstant>0.06</momentConstant>
+          <timeConstantUp>0.0125</timeConstantUp>
+          <timeConstantDown>0.025</timeConstantDown>
+          <maxRotVelocity>838</maxRotVelocity>
+        </rotor>
+      </rotors>
+    </plugin>
+  </gazebo>
+  <!-- â”€â”€â”€ GZ: POSE PUBLISHER â”€â”€â”€ -->
+  <gazebo>
+    <plugin filename="gz-sim-pose-publisher-system"
+            name="gz::sim::systems::PosePublisher">
+      <publish_link_pose>true</publish_link_pose>
+      <publish_nested_model_pose>false</publish_nested_model_pose>
+      <update_rate>50</update_rate>
+    </plugin>
+  </gazebo>
+  <!-- â”€â”€â”€ GZ: ODOMETRY PUBLISHER â”€â”€â”€ -->
+  <gazebo>
+    <plugin filename="gz-sim-odometry-publisher-system"
+            name="gz::sim::systems::OdometryPublisher">
+      <odom_frame>odom</odom_frame>
+      <robot_base_frame>base_link</robot_base_frame>
+      <update_frequency>50</update_frequency>
+      <gaussian_noise>0.001</gaussian_noise>
+      <xyz_offset>0 0 0</xyz_offset>
+      <rpy_offset>0 0 0</rpy_offset>
     </plugin>
   </gazebo>
