Commit message: Build files and .xarco files

File: ControlSystemsPipeline/tranq_ws/src/tranq_description/urdf/drone.urdf.xacro (robot description, xacro)
@@ -1,18 +1,16 @@
 <?xml version="1.0"?>
 <robot xmlns:xacro="http://www.ros.org/wiki/xacro" name="tranq_drone">
-  <!-- â”€â”€â”€ MATERIALS â”€â”€â”€ -->
+  <!-- MATERIALS -->
   <material name="dark_grey"><color rgba="0.15 0.15 0.15 1.0"/></material>
   <material name="orange">   <color rgba="0.9  0.4  0.0  1.0"/></material>
   <material name="black">    <color rgba="0.05 0.05 0.05 1.0"/></material>
-  <!-- â”€â”€â”€ BASE LINK (FRAME) â”€â”€â”€ -->
+  <!-- BASE LINK -->
   <link name="base_link">
     <inertial>
       <mass value="2.5"/>
       <origin xyz="0 0 0" rpy="0 0 0"/>
-      <!-- Corrected inertia tensor for X-frame quadrotor: arm_len=0.25m -->
       <inertia ixx="0.0347" ixy="0.0" ixz="0.0"
                iyy="0.0347" iyz="0.0" izz="0.0630"/>
     </inertial>
-    <!-- X-arm 1 -->
     <visual>
       <origin xyz="0 0 0" rpy="0 0 0.785"/>
@@ -20,5 +18,4 @@
       <material name="dark_grey"/>
     </visual>
-    <!-- X-arm 2 -->
     <visual>
       <origin xyz="0 0 0" rpy="0 0 -0.785"/>
@@ -26,5 +23,4 @@
       <material name="dark_grey"/>
     </visual>
-    <!-- Center hub -->
     <visual>
       <origin xyz="0 0 0.02" rpy="0 0 0"/>
@@ -32,5 +28,4 @@
       <material name="orange"/>
     </visual>
-    <!-- Dart launcher barrel -->
     <visual>
       <origin xyz="0.20 0 -0.04" rpy="0 1.5708 0"/>
@@ -38,5 +33,4 @@
       <material name="black"/>
     </visual>
-    <!-- Landing legs -->
     <visual>
       <origin xyz=" 0.12  0.12 -0.085" rpy="0 0 0"/>
@@ -64,10 +58,6 @@
     </collision>
   </link>
-  <!-- â”€â”€â”€ MOTOR / ROTOR MACRO â”€â”€â”€ -->
-  <!-- FIX: joints are now 'revolute' (not 'fixed') so the
-       MulticopterMotorModel plugin can apply thrust forces.
-       Previously this was 'fixed' which meant the physics
-       system saw zero rotor inertia change = no thrust. -->
-  <xacro:macro name="motor_link" params="name x y direction">
+  <!-- MOTOR / ROTOR MACRO -->
+  <xacro:macro name="motor_link" params="name x y direction motor_number">
     <link name="${name}">
       <inertial>
@@ -92,13 +82,10 @@
       </collision>
     </link>
-    <joint name="${name}_joint" type="revolute">
+    <joint name="${name}_joint" type="continuous">
       <parent link="base_link"/>
       <child link="${name}"/>
       <origin xyz="${x} ${y} 0.03" rpy="0 0 0"/>
       <axis xyz="0 0 1"/>
-      <!-- Effectively unlimited rotation for propellers -->
-      <limit lower="-1e6" upper="1e6" effort="10" velocity="3500"/>
     </joint>
-    <!-- Gz Harmonic MulticopterMotorModel plugin per rotor -->
     <gazebo>
       <plugin filename="gz-sim-multicopter-motor-model-system"
@@ -114,5 +101,5 @@
         <momentConstant>0.06</momentConstant>
         <commandSubTopic>gazebo/command/motor_speed</commandSubTopic>
-        <motorNumber>0</motorNumber>
+        <motorNumber>${motor_number}</motorNumber>
         <rotorDragCoefficient>8.06428e-05</rotorDragCoefficient>
         <rollingMomentCoefficient>1e-06</rollingMomentCoefficient>
@@ -122,23 +109,19 @@
     </gazebo>
   </xacro:macro>
-  <!-- FIX: CCW on FL/RR, CW on FR/RL for correct yaw authority -->
-  <xacro:motor_link name="rotor_fl" x=" 0.177" y=" 0.177" direction="ccw"/>
-  <xacro:motor_link name="rotor_fr" x=" 0.177" y="-0.177" direction="cw"/>
-  <xacro:motor_link name="rotor_rl" x="-0.177" y=" 0.177" direction="cw"/>
-  <xacro:motor_link name="rotor_rr" x="-0.177" y="-0.177" direction="ccw"/>
-  <!-- â”€â”€â”€ INCLUDE SENSORS â”€â”€â”€ -->
+  <xacro:motor_link name="rotor_fl" x=" 0.177" y=" 0.177" direction="ccw" motor_number="0"/>
+  <xacro:motor_link name="rotor_fr" x=" 0.177" y="-0.177" direction="cw"  motor_number="1"/>
+  <xacro:motor_link name="rotor_rl" x="-0.177" y=" 0.177" direction="cw"  motor_number="2"/>
+  <xacro:motor_link name="rotor_rr" x="-0.177" y="-0.177" direction="ccw" motor_number="3"/>
+  <!-- SENSORS -->
   <xacro:include filename="$(find tranq_description)/urdf/sensors.urdf.xacro"/>
   <xacro:camera_sensor parent="base_link"/>
   <xacro:imu_sensor parent="base_link"/>
-  <!-- â”€â”€â”€ FIX: MulticopterVelocityControl â€” THIS WAS COMPLETELY MISSING â”€â”€â”€ -->
-  <!-- This plugin translates /cmd_vel Twist into per-motor speed commands.
-       Without it the drone has no relationship between ROS velocity commands
-       and Gazebo physics â€” it simply falls through the world. -->
+  <!-- MulticopterVelocityControl — Gz8 schema -->
   <gazebo>
     <plugin filename="gz-sim-multicopter-control-system"
             name="gz::sim::systems::MulticopterVelocityControl">
       <robotNamespace>tranq_drone</robotNamespace>
-      <commandSubTopic>/cmd_vel</commandSubTopic>
-      <enableSubTopic>/enable_motors</enableSubTopic>
+      <commandSubTopic>cmd_vel</commandSubTopic>
+      <enableSubTopic>enable_motors</enableSubTopic>
       <comLinkName>base_link</comLinkName>
       <velocityGain>2.7 2.7 2.7</velocityGain>
@@ -146,14 +129,11 @@
       <angularRateGain>0.4 0.4 0.12</angularRateGain>
       <maximumLinearAcceleration>2 2 2</maximumLinearAcceleration>
-      <rotors>
+      <rotorConfiguration>
         <rotor>
           <jointName>rotor_fl_joint</jointName>
           <bodyFrame>rotor_fl</bodyFrame>
           <direction>1</direction>
-          <motorConstant>8.54858e-06</motorConstant>
+          <forceConstant>8.54858e-06</forceConstant>
           <momentConstant>0.06</momentConstant>
-          <timeConstantUp>0.0125</timeConstantUp>
-          <timeConstantDown>0.025</timeConstantDown>
-          <maxRotVelocity>838</maxRotVelocity>
         </rotor>
         <rotor>
@@ -161,9 +141,6 @@
           <bodyFrame>rotor_fr</bodyFrame>
           <direction>-1</direction>
-          <motorConstant>8.54858e-06</motorConstant>
+          <forceConstant>8.54858e-06</forceConstant>
           <momentConstant>0.06</momentConstant>
-          <timeConstantUp>0.0125</timeConstantUp>
-          <timeConstantDown>0.025</timeConstantDown>
-          <maxRotVelocity>838</maxRotVelocity>
         </rotor>
         <rotor>
@@ -171,9 +148,6 @@
           <bodyFrame>rotor_rl</bodyFrame>
           <direction>-1</direction>
-          <motorConstant>8.54858e-06</motorConstant>
+          <forceConstant>8.54858e-06</forceConstant>
           <momentConstant>0.06</momentConstant>
-          <timeConstantUp>0.0125</timeConstantUp>
-          <timeConstantDown>0.025</timeConstantDown>
-          <maxRotVelocity>838</maxRotVelocity>
         </rotor>
         <rotor>
@@ -181,14 +155,11 @@
           <bodyFrame>rotor_rr</bodyFrame>
           <direction>1</direction>
-          <motorConstant>8.54858e-06</motorConstant>
+          <forceConstant>8.54858e-06</forceConstant>
           <momentConstant>0.06</momentConstant>
-          <timeConstantUp>0.0125</timeConstantUp>
-          <timeConstantDown>0.025</timeConstantDown>
-          <maxRotVelocity>838</maxRotVelocity>
         </rotor>
-      </rotors>
+      </rotorConfiguration>
     </plugin>
   </gazebo>
-  <!-- â”€â”€â”€ GZ: POSE PUBLISHER â”€â”€â”€ -->
+  <!-- POSE PUBLISHER -->
   <gazebo>
     <plugin filename="gz-sim-pose-publisher-system"
@@ -199,5 +170,5 @@
     </plugin>
   </gazebo>
-  <!-- â”€â”€â”€ GZ: ODOMETRY PUBLISHER â”€â”€â”€ -->
+  <!-- ODOMETRY PUBLISHER -->
   <gazebo>
     <plugin filename="gz-sim-odometry-publisher-system"

Commit message: Copied source branch code

File: ControlSystemsPipeline/tranq_ws/src/tranq_description/urdf/drone.urdf.xacro (robot description, xacro)
@@ -1,183 +1,31 @@
 <?xml version="1.0"?>
 <robot xmlns:xacro="http://www.ros.org/wiki/xacro" name="tranq_drone">
-  <!-- MATERIALS -->
-  <material name="dark_grey"><color rgba="0.15 0.15 0.15 1.0"/></material>
-  <material name="orange">   <color rgba="0.9  0.4  0.0  1.0"/></material>
-  <material name="black">    <color rgba="0.05 0.05 0.05 1.0"/></material>
-  <!-- BASE LINK -->
+  <xacro:include filename="$(find tranq_description)/urdf/sensors.urdf.xacro"/>
   <link name="base_link">
     <inertial>
-      <mass value="2.5"/>
       <origin xyz="0 0 0" rpy="0 0 0"/>
-      <inertia ixx="0.0347" ixy="0.0" ixz="0.0"
-               iyy="0.0347" iyz="0.0" izz="0.0630"/>
+      <mass value="1.5"/>
+      <inertia ixx="0.03" ixy="0.0" ixz="0.0" iyy="0.03" iyz="0.0" izz="0.05"/>
     </inertial>
     <visual>
-      <origin xyz="0 0 0" rpy="0 0 0.785"/>
-      <geometry><box size="0.50 0.08 0.06"/></geometry>
-      <material name="dark_grey"/>
-    </visual>
-    <visual>
-      <origin xyz="0 0 0" rpy="0 0 -0.785"/>
-      <geometry><box size="0.50 0.08 0.06"/></geometry>
-      <material name="dark_grey"/>
-    </visual>
-    <visual>
-      <origin xyz="0 0 0.02" rpy="0 0 0"/>
-      <geometry><cylinder radius="0.09" length="0.08"/></geometry>
-      <material name="orange"/>
-    </visual>
-    <visual>
-      <origin xyz="0.20 0 -0.04" rpy="0 1.5708 0"/>
-      <geometry><cylinder radius="0.025" length="0.18"/></geometry>
-      <material name="black"/>
-    </visual>
-    <visual>
-      <origin xyz=" 0.12  0.12 -0.085" rpy="0 0 0"/>
-      <geometry><cylinder radius="0.01" length="0.14"/></geometry>
-      <material name="dark_grey"/>
-    </visual>
-    <visual>
-      <origin xyz="-0.12  0.12 -0.085" rpy="0 0 0"/>
-      <geometry><cylinder radius="0.01" length="0.14"/></geometry>
-      <material name="dark_grey"/>
-    </visual>
-    <visual>
-      <origin xyz=" 0.12 -0.12 -0.085" rpy="0 0 0"/>
-      <geometry><cylinder radius="0.01" length="0.14"/></geometry>
-      <material name="dark_grey"/>
-    </visual>
-    <visual>
-      <origin xyz="-0.12 -0.12 -0.085" rpy="0 0 0"/>
-      <geometry><cylinder radius="0.01" length="0.14"/></geometry>
-      <material name="dark_grey"/>
+      <origin xyz="0 0 0" rpy="0 0 0"/>
+      <geometry><box size="0.35 0.35 0.08"/></geometry>
+      <material name="dark_grey"><color rgba="0.2 0.2 0.2 1"/></material>
     </visual>
     <collision>
       <origin xyz="0 0 0" rpy="0 0 0"/>
-      <geometry><box size="0.58 0.58 0.14"/></geometry>
+      <geometry><box size="0.35 0.35 0.08"/></geometry>
     </collision>
   </link>
-  <!-- MOTOR / ROTOR MACRO -->
-  <xacro:macro name="motor_link" params="name x y direction motor_number">
-    <link name="${name}">
-      <inertial>
-        <mass value="0.05"/>
-        <origin xyz="0 0 0" rpy="0 0 0"/>
-        <inertia ixx="1e-5" ixy="0" ixz="0"
-                 iyy="1e-5" iyz="0" izz="9.75e-6"/>
-      </inertial>
-      <visual>
-        <origin xyz="0 0 0.02" rpy="0 0 0"/>
-        <geometry><cylinder radius="0.025" length="0.05"/></geometry>
-        <material name="black"/>
-      </visual>
-      <visual>
-        <origin xyz="0 0 0.055" rpy="0 0 0"/>
-        <geometry><cylinder radius="0.115" length="0.004"/></geometry>
-        <material name="dark_grey"/>
-      </visual>
-      <collision>
-        <origin xyz="0 0 0.055" rpy="0 0 0"/>
-        <geometry><cylinder radius="0.115" length="0.01"/></geometry>
-      </collision>
-    </link>
-    <joint name="${name}_joint" type="continuous">
-      <parent link="base_link"/>
-      <child link="${name}"/>
-      <origin xyz="${x} ${y} 0.03" rpy="0 0 0"/>
-      <axis xyz="0 0 1"/>
-    </joint>
-    <gazebo>
-      <plugin filename="gz-sim-multicopter-motor-model-system"
-              name="gz::sim::systems::MulticopterMotorModel">
-        <robotNamespace>tranq_drone</robotNamespace>
-        <jointName>${name}_joint</jointName>
-        <linkName>${name}</linkName>
-        <turningDirection>${direction}</turningDirection>
-        <timeConstantUp>0.0125</timeConstantUp>
-        <timeConstantDown>0.025</timeConstantDown>
-        <maxRotVelocity>838.0</maxRotVelocity>
-        <motorConstant>8.54858e-06</motorConstant>
-        <momentConstant>0.06</momentConstant>
-        <commandSubTopic>gazebo/command/motor_speed</commandSubTopic>
-        <motorNumber>${motor_number}</motorNumber>
-        <rotorDragCoefficient>8.06428e-05</rotorDragCoefficient>
-        <rollingMomentCoefficient>1e-06</rollingMomentCoefficient>
-        <rotorVelocitySlowdownSim>10</rotorVelocitySlowdownSim>
-        <motorType>velocity</motorType>
-      </plugin>
-    </gazebo>
-  </xacro:macro>
-  <xacro:motor_link name="rotor_fl" x=" 0.177" y=" 0.177" direction="ccw" motor_number="0"/>
-  <xacro:motor_link name="rotor_fr" x=" 0.177" y="-0.177" direction="cw"  motor_number="1"/>
-  <xacro:motor_link name="rotor_rl" x="-0.177" y=" 0.177" direction="cw"  motor_number="2"/>
-  <xacro:motor_link name="rotor_rr" x="-0.177" y="-0.177" direction="ccw" motor_number="3"/>
-  <!-- SENSORS -->
-  <xacro:include filename="$(find tranq_description)/urdf/sensors.urdf.xacro"/>
   <xacro:camera_sensor parent="base_link"/>
-  <xacro:imu_sensor parent="base_link"/>
-  <!-- MulticopterVelocityControl — Gz8 schema -->
+  <xacro:tof_sensor parent="base_link"
+    name="tof_center" topic="/range_1"
+    xyz="0.15 0.0 -0.02" rpy="0 1.5708 0"/>
+  <xacro:tof_sensor parent="base_link"
+    name="tof_offset" topic="/range_2"
+    xyz="0.15 0.0 -0.12" rpy="0 1.5708 0"/>
   <gazebo>
-    <plugin filename="gz-sim-multicopter-control-system"
-            name="gz::sim::systems::MulticopterVelocityControl">
-      <robotNamespace>tranq_drone</robotNamespace>
-      <commandSubTopic>cmd_vel</commandSubTopic>
-      <enableSubTopic>enable_motors</enableSubTopic>
-      <comLinkName>base_link</comLinkName>
-      <velocityGain>2.7 2.7 2.7</velocityGain>
-      <attitudeGain>3.0 3.0 0.15</attitudeGain>
-      <angularRateGain>0.4 0.4 0.12</angularRateGain>
-      <maximumLinearAcceleration>2 2 2</maximumLinearAcceleration>
-      <rotorConfiguration>
-        <rotor>
-          <jointName>rotor_fl_joint</jointName>
-          <bodyFrame>rotor_fl</bodyFrame>
-          <direction>1</direction>
-          <forceConstant>8.54858e-06</forceConstant>
-          <momentConstant>0.06</momentConstant>
-        </rotor>
-        <rotor>
-          <jointName>rotor_fr_joint</jointName>
-          <bodyFrame>rotor_fr</bodyFrame>
-          <direction>-1</direction>
-          <forceConstant>8.54858e-06</forceConstant>
-          <momentConstant>0.06</momentConstant>
-        </rotor>
-        <rotor>
-          <jointName>rotor_rl_joint</jointName>
-          <bodyFrame>rotor_rl</bodyFrame>
-          <direction>-1</direction>
-          <forceConstant>8.54858e-06</forceConstant>
-          <momentConstant>0.06</momentConstant>
-        </rotor>
-        <rotor>
-          <jointName>rotor_rr_joint</jointName>
-          <bodyFrame>rotor_rr</bodyFrame>
-          <direction>1</direction>
-          <forceConstant>8.54858e-06</forceConstant>
-          <momentConstant>0.06</momentConstant>
-        </rotor>
-      </rotorConfiguration>
-    </plugin>
-  </gazebo>
-  <!-- POSE PUBLISHER -->
-  <gazebo>
-    <plugin filename="gz-sim-pose-publisher-system"
-            name="gz::sim::systems::PosePublisher">
-      <publish_link_pose>true</publish_link_pose>
-      <publish_nested_model_pose>false</publish_nested_model_pose>
-      <update_rate>50</update_rate>
-    </plugin>
-  </gazebo>
-  <!-- ODOMETRY PUBLISHER -->
-  <gazebo>
-    <plugin filename="gz-sim-odometry-publisher-system"
-            name="gz::sim::systems::OdometryPublisher">
-      <odom_frame>odom</odom_frame>
-      <robot_base_frame>base_link</robot_base_frame>
-      <update_frequency>50</update_frequency>
-      <gaussian_noise>0.001</gaussian_noise>
-      <xyz_offset>0 0 0</xyz_offset>
-      <rpy_offset>0 0 0</rpy_offset>
+    <plugin name="gazebo_ros_control" filename="libgazebo_ros_control.so">
+      <robotNamespace>/tranq_drone</robotNamespace>
     </plugin>
   </gazebo>

File: ControlSystemsPipeline/tranq_ws/src/tranq_description/urdf/sensors.urdf.xacro (robot description, xacro)
@@ -1,41 +1,19 @@
 <?xml version="1.0"?>
 <robot xmlns:xacro="http://www.ros.org/wiki/xacro">
-  <!-- â•â•â•â•â•â•â•â•â•â•â•â•â•â•â• FRONT CAMERA â•â•â•â•â•â•â•â•â•â•â•â•â•â•â• -->
-  <!-- FIX: Added inertial block (was missing, causing URDF parse errors).
-       Added optical frame joint (required for ROS image_transport / camera_info).
-       Added camera distortion model matching training data collection setup.
-       Camera tilted 15Â° downward for target visibility during approach. -->
   <xacro:macro name="camera_sensor" params="parent">
     <link name="camera_link">
-      <inertial>
-        <mass value="0.035"/>
-        <inertia ixx="1e-6" ixy="0" ixz="0"
-                 iyy="1e-6" iyz="0" izz="1e-6"/>
-      </inertial>
       <visual>
-        <geometry><box size="0.04 0.06 0.03"/></geometry>
-        <material name="black"><color rgba="0.05 0.05 0.05 1"/></material>
+        <geometry><box size="0.03 0.05 0.03"/></geometry>
+        <material name="black"><color rgba="0 0 0 1"/></material>
       </visual>
-      <collision>
-        <geometry><box size="0.04 0.06 0.03"/></geometry>
-      </collision>
     </link>
     <joint name="camera_joint" type="fixed">
       <parent link="${parent}"/>
       <child link="camera_link"/>
-      <!-- 15-degree downward pitch for target tracking during hover -->
-      <origin xyz="0.22 0 -0.02" rpy="0 0.2618 0"/>
-    </joint>
-    <!-- FIX: Optical frame required by ROS image_transport convention -->
-    <link name="camera_optical_link"/>
-    <joint name="camera_optical_joint" type="fixed">
-      <parent link="camera_link"/>
-      <child link="camera_optical_link"/>
-      <origin xyz="0 0 0" rpy="-1.5708 0 -1.5708"/>
+      <origin xyz="0.18 0 -0.01" rpy="0 0 0"/>
     </joint>
     <gazebo reference="camera_link">
       <sensor name="front_camera" type="camera">
         <update_rate>30</update_rate>
-        <always_on>true</always_on>
         <camera>
           <horizontal_fov>1.3962634</horizontal_fov>
@@ -43,61 +21,47 @@
             <width>640</width>
             <height>480</height>
-            <format>R8G8B8</format>
+            <format>RGB_INT8</format>
           </image>
-          <clip>
-            <near>0.1</near>
-            <far>300</far>
-          </clip>
-          <noise>
-            <type>gaussian</type>
-            <mean>0.0</mean>
-            <stddev>0.007</stddev>
-          </noise>
-          <!-- FIX: Distortion model added to match real sensor characteristics -->
-          <distortion>
-            <k1>-0.25</k1><k2>0.12</k2><k3>0.0</k3>
-            <p1>-0.00028</p1><p2>-0.00005</p2>
-            <center>0.5 0.5</center>
-          </distortion>
+          <clip><near>0.1</near><far>100.0</far></clip>
+          <noise><type>gaussian</type><mean>0.0</mean><stddev>0.005</stddev></noise>
         </camera>
         <topic>/camera/image_raw</topic>
-        <gz_frame_id>camera_optical_link</gz_frame_id>
+        <gz_frame_id>camera_link</gz_frame_id>
       </sensor>
     </gazebo>
   </xacro:macro>
-  <!-- â•â•â•â•â•â•â•â•â•â•â•â•â•â•â• IMU SENSOR â•â•â•â•â•â•â•â•â•â•â•â•â•â•â• -->
-  <!-- FIX: IMU was completely missing from original sensors.urdf.xacro.
-       Required for odometry, EKF, and altitude hold. Noise parameters
-       modelled on MPU-6000 datasheet. -->
-  <xacro:macro name="imu_sensor" params="parent">
-    <link name="imu_link">
-      <inertial>
-        <mass value="0.015"/>
-        <inertia ixx="1e-7" ixy="0" ixz="0"
-                 iyy="1e-7" iyz="0" izz="1e-7"/>
-      </inertial>
+  <xacro:macro name="tof_sensor" params="parent name topic xyz rpy">
+    <link name="${name}_link">
+      <visual>
+        <geometry><box size="0.01 0.01 0.01"/></geometry>
+        <material name="silver"><color rgba="0.8 0.8 0.8 1"/></material>
+      </visual>
     </link>
-    <joint name="imu_joint" type="fixed">
+    <joint name="${name}_joint" type="fixed">
       <parent link="${parent}"/>
-      <child link="imu_link"/>
-      <origin xyz="0 0 0" rpy="0 0 0"/>
+      <child link="${name}_link"/>
+      <origin xyz="${xyz}" rpy="${rpy}"/>
     </joint>
-    <gazebo reference="imu_link">
-      <sensor name="imu_sensor" type="imu">
-        <update_rate>400</update_rate>
-        <always_on>true</always_on>
-        <imu>
-          <angular_velocity>
-            <x><noise type="gaussian"><mean>0</mean><stddev>2e-4</stddev></noise></x>
-            <y><noise type="gaussian"><mean>0</mean><stddev>2e-4</stddev></noise></y>
-            <z><noise type="gaussian"><mean>0</mean><stddev>2e-4</stddev></noise></z>
-          </angular_velocity>
-          <linear_acceleration>
-            <x><noise type="gaussian"><mean>0</mean><stddev>1.7e-2</stddev></noise></x>
-            <y><noise type="gaussian"><mean>0</mean><stddev>1.7e-2</stddev></noise></y>
-            <z><noise type="gaussian"><mean>0</mean><stddev>1.7e-2</stddev></noise></z>
-          </linear_acceleration>
-        </imu>
-        <topic>/imu</topic>
+    <gazebo reference="${name}_link">
+      <sensor name="${name}" type="gpu_lidar">
+        <update_rate>30</update_rate>
+        <lidar>
+          <scan>
+            <horizontal>
+              <samples>1</samples>
+              <resolution>1</resolution>
+              <min_angle>0</min_angle>
+              <max_angle>0</max_angle>
+            </horizontal>
+          </scan>
+          <range>
+            <min>0.05</min>
+            <max>30.0</max>
+            <resolution>0.01</resolution>
+          </range>
+          <noise><type>gaussian</type><mean>0.0</mean><stddev>0.02</stddev></noise>
+        </lidar>
+        <topic>${topic}</topic>
+        <gz_frame_id>${name}_link</gz_frame_id>
       </sensor>
     </gazebo>
